Commit message: Add interactive dual-arm planning, swerve drive, and rendering fixes
- interactive_plan.py: full swerve-drive base control (WASD + turn), dual-arm
  CuRobo motion planning, lift joint, ghost trajectory preview, ROS 2 cmd_vel
  publishing, GLFW key intercept to prevent W/S/D rendering shortcut conflicts
- scene_ffw_sg2.xml: split floor (physics z=0 invisible, visual z=-25 mm) to
  eliminate wheel-mesh z-fighting during rotation
- ffw_sg2.xml: robot model refinements
- ffw_sg2_left_arm.yml: updated CuRobo config for left arm
- curobo_server.py: server improvements for dual-arm support
- docker: updated Dockerfile and compose for new dependencies
- ffw_sg2_follower.urdf: URDF corrections

Co-Authored-By: Claude Sonnet 4.6 <noreply@anthropic.com>

File: robot/urdf/urdf/ffw_sg2_rev1_follower/ffw_sg2_follower.urdf (robot description, URDF)
Before this commit: robot ffw_sg2_follower, 40 links, 39 joints
Links:
- added link arm_l_tcp
- added link arm_r_tcp
Joints:
- added joint arm_l_tcp_joint: type fixed, parent arm_l_link7, child arm_l_tcp, origin xyz=0 0 -0.215 rpy=0 0 0
- added joint arm_r_tcp_joint: type fixed, parent arm_r_link7, child arm_r_tcp, origin xyz=0 0 -0.215 rpy=0 0 0
